File: hw/sch_pcb/CCP2019V01.kicad_pcb (KiCad board)
At the start: 2 copper layers, 90.9 x 50.3 mm, 111 parts, among them J1 HEADER_2x01_PARALLEL, J19 HEADER_2x01_PARALLEL, J2 HEADER_2x01_PARALLEL, J22 HEADER_2x03, J3 HEADER_2x01_PARALLEL, J4 HEADER_1x01, J5 HEADER_1x01, J6 HEADER_1x01, J7 HEADER_1x01, M1 HOLE, M2 HOLE, M3 HOLE, M4 HOLE, M6 BMI-S-210-F, M7 BMI-S-210-F, U1 OPA2314, U10 ATMEGA1284P-AU, U11 PCF85263A, U2 OPA2314, U3 ISL21080DIH312Z-TK 1V25, U4 TS7211, U5 TS5A4594, U6 TPS613221ADBV, U8 TPS613222ADBV, Y1 16MHz, Y2 ABS07-120-32.768KHZ-T

Commit message: Convert to KiCADv7 project.
Other:
- net class Default removed
- net class MLAB_default removed
- net class MLAB_power removed
